File: board/prototype/ethernet2serial/ethernet2serial.kicad_pcb (KiCad board)
At the start: 2 copper layers, 20 x 33.3 mm, 23 parts, among them J2 J1B1211CCD, J3 Conn_01x05, J4 Conn_01x05, U1 ATtiny1606-M, U2 ENC28J60x-ML, Y1 XRCGB25M000F0L00R0

Commit message: Improving readme
Other:
- net class Default removed
